File: hardware/hat/kingfisher-hat.kicad_pcb (KiCad board)
At the start: 4 copper layers, 65 x 56 mm, 17 parts, among them J1 GPIO, J2 U.FL, U1 ICM-45686, U2 BMP581, U3 AP2112K-3.3, U4 NEO-M9N

Commit message: feat(hat): route rev 0.3 on the JLC04161H-7628 stack
The RF width is 0.32 mm for the pressed 7.1 mil outer dielectric, and the ground pours stitch SMD islands into the inner planes.

Co-authored-by: Cursor <cursoragent@cursor.com>
Parts:
- added BT1: CR2032, BatteryHolder_Keystone_3002_1x2032, F.Cu at (124.0, 83.0)
- added BT2: ML414H, ML414H, F.Cu at (125.0, 66.0)
- added C10: 47pF, C_0402_1005Metric, F.Cu at (160.0, 60.5)
- added C11: 100nF, C_0402_1005Metric, F.Cu at (125.5, 58.0)
- added C8: 100nF, C_0402_1005Metric, F.Cu at (136.2, 61.8)
- added C9: 1uF, C_0603_1608Metric, F.Cu at (130.2, 64.2)
- added D1: PMEG4005EJ, D_SOD-323F, F.Cu at (134.5, 64.2)
- added D2: Green, LED_0603_1608Metric, F.Cu at (133.8, 67.8)
- added FB1: 120R, L_0402_1005Metric, F.Cu at (157.7, 57.0)
- added J3: X1200, PinHeader_1x05_P2.54mm_Horizontal, F.Cu at (153.5, 78.0)
- added R1: 33, R_0603_1608Metric, F.Cu at (139.2, 63.5)
- added R2: 33, R_0603_1608Metric, F.Cu at (139.2, 67.6)
- added R3: 10k, R_0402_1005Metric, F.Cu at (158.2, 66.5)
- added R4: 1k, R_0603_1608Metric, F.Cu at (130.2, 68.0)
- added R5: 33, R_0402_1005Metric, F.Cu at (157.4, 59.7)
- added R6: 1k, R_0603_1608Metric, F.Cu at (137.0, 67.8)
- added R7: 4.7k, R_0402_1005Metric, F.Cu at (119.6, 64.6)
- added R8: 4.7k, R_0402_1005Metric, F.Cu at (119.6, 67.0)
- added TP1: +3V3, TestPoint_Pad_D1.5mm, F.Cu at (109.0, 53.3)
- added TP10: GPS_PPS, TestPoint_Pad_D1.5mm, F.Cu at (149.2, 81.2)
- added TP11: IMU_INT, TestPoint_Pad_D1.5mm, F.Cu at (149.2, 84.4)
- added TP12: GND, TestPoint_Pad_D1.5mm, F.Cu at (149.2, 87.6)
- added TP2: +5V, TestPoint_Pad_D1.5mm, F.Cu at (112.3, 53.3)
- added TP3: +3V3_GPS, TestPoint_Pad_D1.5mm, F.Cu at (115.6, 53.3)
- added TP4: V_BCKP, TestPoint_Pad_D1.5mm, F.Cu at (118.9, 53.3)
- added TP5: VBAT, TestPoint_Pad_D1.5mm, F.Cu at (122.2, 53.3)
- added TP6: SDA, TestPoint_Pad_D1.5mm, F.Cu at (125.5, 53.3)
- added TP7: SCL, TestPoint_Pad_D1.5mm, F.Cu at (128.8, 53.3)
- added TP8: UART_TX, TestPoint_Pad_D1.5mm, F.Cu at (132.1, 53.3)
- added TP9: UART_RX, TestPoint_Pad_D1.5mm, F.Cu at (149.2, 78.0)
- added U5: RV-3028-C7, MicroCrystal_C7_SON-8_1.5x3.2mm_P0.9mm, F.Cu at (121.5, 58.0)
- C5, C6: footprint C_0402_1005Metric -> C_0603_1608Metric
- U1: footprint Bosch_LGA-14_3x2.5mm_P0.5mm -> ICM-45686
- moved U2 48.5 mm to (112.0, 65.5)
- moved C4 45.4 mm to (116.5, 66.6)
- moved C3 40.8 mm to (116.5, 64.8)
- moved C2 29.2 mm to (116.5, 59.4)
- moved U1 27.7 mm to (112.0, 58.0)
- moved C1 25.5 mm to (116.5, 57.2)
- moved C5 19.2 mm to (136.2, 56.6)
- moved U4 17.1 mm to (148.5, 61.5), turned to 180 degrees
- moved C6 13.4 mm to (136.2, 59.2)
- moved U3 10.7 mm to (130.5, 58.0)
- moved C7 7.47 mm to (139.4, 58.0)
- moved J2 6.23 mm to (161.2, 55.6)
Connections:
- C1 pad 1: (no net) -> +3V3
- C1 pad 2: (no net) -> GND
- C2 pad 1: (no net) -> +3V3
- C2 pad 2: (no net) -> GND
- C3 pad 1: (no net) -> +3V3
- C3 pad 2: (no net) -> GND
- C4 pad 1: (no net) -> +3V3
- C4 pad 2: (no net) -> GND
- C5 pad 1: (no net) -> +5V
- C5 pad 2: (no net) -> GND
- C6 pad 1: (no net) -> +3V3_GPS
- C6 pad 2: (no net) -> GND
- C7 pad 1: (no net) -> +3V3_GPS
- C7 pad 2: (no net) -> GND
- J1 pad 10: /GPIO15/RXD0 -> UART_RX
- J1 pad 11: /GPIO17 -> IMU_INT
- J1 pad 12: /GPIO18/PCM.CLK -> GPS_PPS
- J1 pad 13: /GPIO27 -> unconnected-(J1-Pin_13-Pad13)
- J1 pad 15: /GPIO22 -> unconnected-(J1-Pin_15-Pad15)
- J1 pad 16: /GPIO23 -> unconnected-(J1-Pin_16-Pad16)
- J1 pad 18: /GPIO24 -> unconnected-(J1-Pin_18-Pad18)
- J1 pad 19: /GPIO10/SPI0.MOSI -> unconnected-(J1-Pin_19-Pad19)
- J1 pad 21: /GPIO9/SPI0.MISO -> unconnected-(J1-Pin_21-Pad21)
- J1 pad 22: /GPIO25 -> unconnected-(J1-Pin_22-Pad22)
- J1 pad 23: /GPIO11/SPI0.SCLK -> unconnected-(J1-Pin_23-Pad23)
- J1 pad 24: /GPIO8/SPI0.CE0 -> unconnected-(J1-Pin_24-Pad24)
- J1 pad 26: /GPIO7/SPI0.CE1 -> unconnected-(J1-Pin_26-Pad26)
- J1 pad 27: /ID_SDA -> unconnected-(J1-Pin_27-Pad27)
- J1 pad 28: /ID_SCL -> unconnected-(J1-Pin_28-Pad28)
- J1 pad 29: /GPIO5 -> unconnected-(J1-Pin_29-Pad29)
- J1 pad 3: /GPIO2/SDA1 -> SDA
- J1 pad 31: /GPIO6 -> PLD
- J1 pad 32: /GPIO12/PWM0 -> unconnected-(J1-Pin_32-Pad32)
- J1 pad 33: /GPIO13/PWM1 -> unconnected-(J1-Pin_33-Pad33)
- J1 pad 35: /GPIO19/PCM.FS -> unconnected-(J1-Pin_35-Pad35)
- J1 pad 36: /GPIO16 -> unconnected-(J1-Pin_36-Pad36)
- J1 pad 37: /GPIO26 -> unconnected-(J1-Pin_37-Pad37)
- J1 pad 38: /GPIO20/PCM.DIN -> unconnected-(J1-Pin_38-Pad38)
- J1 pad 40: /GPIO21/PCM.DOUT -> unconnected-(J1-Pin_40-Pad40)
- J1 pad 5: /GPIO3/SCL1 -> SCL
- J1 pad 7: /GPIO4/GPCLK0 -> unconnected-(J1-Pin_7-Pad7)
- J1 pad 8: /GPIO14/TXD0 -> UART_TX
- J2 pad 1: (no net) -> RF
- J2 pad 2: (no net) -> GND
- U1 pad 1: (no net) -> GND
- U1 pad 10: (no net) -> unconnected-(U1-NC-Pad10)
- U1 pad 11: (no net) -> unconnected-(U1-NC-Pad11)
- U1 pad 12: (no net) -> +3V3
- U1 pad 13: (no net) -> SCL
- U1 pad 14: (no net) -> SDA
- U1 pad 2: (no net) -> unconnected-(U1-NC-Pad2)
- U1 pad 3: (no net) -> unconnected-(U1-NC-Pad3)
- U1 pad 4: (no net) -> IMU_INT
- U1 pad 5: (no net) -> +3V3
- U1 pad 6: (no net) -> GND
- U1 pad 7: (no net) -> unconnected-(U1-NC-Pad7)
- U1 pad 8: (no net) -> +3V3
- U1 pad 9: (no net) -> unconnected-(U1-INT2-Pad9)
- U2 pad 1: (no net) -> +3V3
- U2 pad 10: (no net) -> +3V3
- U2 pad 2: (no net) -> SCL
- U2 pad 3: (no net) -> GND
- U2 pad 4: (no net) -> SDA
- U2 pad 5: (no net) -> +3V3
- U2 pad 6: (no net) -> +3V3
- U2 pad 7: (no net) -> unconnected-(U2-INT-Pad7)
- U2 pad 8: (no net) -> GND
- U2 pad 9: (no net) -> GND
- U3 pad 1: (no net) -> +5V
- U3 pad 2: (no net) -> GND
- U3 pad 3: (no net) -> +5V
- U3 pad 4: (no net) -> unconnected-(U3-NC-Pad4)
- U3 pad 5: (no net) -> +3V3_GPS
- U4 pad 1: (no net) -> unconnected-(U4-~{SAFEBOOT}-Pad1)
- U4 pad 10: (no net) -> GND
- U4 pad 11: (no net) -> RF
- U4 pad 12: (no net) -> GND
- U4 pad 13: (no net) -> GND
- U4 pad 14: (no net) -> unconnected-(U4-LNA_EN-Pad14)
- U4 pad 15: (no net) -> unconnected-(U4-RESERVED-Pad15)
- U4 pad 16: (no net) -> unconnected-(U4-RESERVED-Pad16)
- U4 pad 17: (no net) -> unconnected-(U4-RESERVED-Pad17)
- U4 pad 18: (no net) -> unconnected-(U4-SDA/~{SPI_CS}-Pad18)
- U4 pad 19: (no net) -> unconnected-(U4-SCL/SPI_CLK-Pad19)
- U4 pad 2: (no net) -> D_SEL
- U4 pad 20: (no net) -> GPS_TX
- U4 pad 21: (no net) -> GPS_RX
- U4 pad 22: (no net) -> V_BCKP
- U4 pad 23: (no net) -> +3V3_GPS
- U4 pad 24: (no net) -> GND
- U4 pad 3: (no net) -> GPS_PPS
- U4 pad 4: (no net) -> unconnected-(U4-EXTINT-Pad4)
- U4 pad 5: (no net) -> unconnected-(U4-USB_DM-Pad5)
- U4 pad 6: (no net) -> unconnected-(U4-USB_DP-Pad6)
- U4 pad 7: (no net) -> +3V3_GPS
- U4 pad 8: (no net) -> unconnected-(U4-~{RESET}-Pad8)
- U4 pad 9: (no net) -> VCC_RF
Routing:
- net +3V3: track 0.00 -> 179.6 mm, vias 0 -> 26
- net +3V3_GPS: track 0.00 -> 117.3 mm, vias 0 -> 12
- net SDA: track 0.00 -> 111.8 mm, vias 0 -> 10
- net SCL: track 0.00 -> 110.5 mm, vias 0 -> 8
- net GPS_PPS: track 0.00 -> 80.0 mm
- net IMU_INT: track 0.00 -> 78.4 mm, vias 0 -> 2
- net UART_RX: track 0.00 -> 70.0 mm, vias 0 -> 4
- net VBAT: track 0.00 -> 61.6 mm, vias 0 -> 7
- net +5V: track 0.00 -> 49.8 mm, vias 0 -> 2
- net V_BCKP: track 0.00 -> 44.3 mm, vias 0 -> 7
- net PLD: track 0.00 -> 44.1 mm
- net UART_TX: track 0.00 -> 41.6 mm
- net CHG: track 0.00 -> 6.70 mm
- net RF: track 0.00 -> 6.62 mm
- net GND: track 0.00 -> 6.31 mm, vias 0 -> 139
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- added copper zone on B.Cu, net GND
- added copper zone on F.Cu, net GND
- added copper zone on In1.Cu, net GND
- added copper zone on In2.Cu, net GND
Other:
- board text added: "rev 0.3"
- board text removed: "KINGFISHER HAT\nICM45686 BMP581 NEO-M9N"
