File: hardware/hat/kingfisher-hat.kicad_sch (KiCad schematic)
At the start: 18 parts, among them J1 GPIO_40, J2 U.FL, U1 ICM-45686, U2 BMP581, U3 AP2112K-3.3, U4 NEO-M9N, U5 RV-3028-C7

Commit message: feat(hat): rebuild the rev 0.3 schematic against the datasheet pins
Rev 0.2 landed power on ground pins. The netlist check is the contract for the GPS, IMU, RTC, and X1200 circuits.

Co-authored-by: Cursor <cursoragent@cursor.com>
Parts:
- removed D2: BAT54, Diode_SMD:D_SOD-123, symbol Device:D_Schottky
- added BT2: ML414H, Kingfisher:ML414H, symbol Device:Battery_Cell
- added C10: 47pF, Capacitor_SMD:C_0402_1005Metric, symbol Device:C
- added C11: 100nF, Capacitor_SMD:C_0402_1005Metric, symbol Device:C
- added C9: 1uF, Capacitor_SMD:C_0603_1608Metric, symbol Device:C
- added D2: Green, LED_SMD:LED_0603_1608Metric, symbol Device:LED
- added FB1: 120R, Inductor_SMD:L_0402_1005Metric, symbol Device:FerriteBead
- added J3: X1200, Connector_PinHeader_2.54mm:PinHeader_1x05_P2.54mm_Horizontal, symbol Connector_Generic:Conn_01x05
- added R1, R2: 33, Resistor_SMD:R_0603_1608Metric, symbol Device:R
- added R3: 10k, Resistor_SMD:R_0402_1005Metric, symbol Device:R
- added R4, R6: 1k, Resistor_SMD:R_0603_1608Metric, symbol Device:R
- added R5: 33, Resistor_SMD:R_0402_1005Metric, symbol Device:R
- added R7, R8: 4.7k, Resistor_SMD:R_0402_1005Metric, symbol Device:R
- added TP1: +3V3, TestPoint:TestPoint_Pad_D1.5mm, symbol Connector:TestPoint
- added TP10: GPS_PPS, TestPoint:TestPoint_Pad_D1.5mm, symbol Connector:TestPoint
- added TP11: IMU_INT, TestPoint:TestPoint_Pad_D1.5mm, symbol Connector:TestPoint
- added TP12: GND, TestPoint:TestPoint_Pad_D1.5mm, symbol Connector:TestPoint
- added TP2: +5V, TestPoint:TestPoint_Pad_D1.5mm, symbol Connector:TestPoint
- added TP3: +3V3_GPS, TestPoint:TestPoint_Pad_D1.5mm, symbol Connector:TestPoint
- added TP4: V_BCKP, TestPoint:TestPoint_Pad_D1.5mm, symbol Connector:TestPoint
- added TP5: VBAT, TestPoint:TestPoint_Pad_D1.5mm, symbol Connector:TestPoint
- added TP6: SDA, TestPoint:TestPoint_Pad_D1.5mm, symbol Connector:TestPoint
- added TP7: SCL, TestPoint:TestPoint_Pad_D1.5mm, symbol Connector:TestPoint
- added TP8: UART_TX, TestPoint:TestPoint_Pad_D1.5mm, symbol Connector:TestPoint
- added TP9: UART_RX, TestPoint:TestPoint_Pad_D1.5mm, symbol Connector:TestPoint
- D1: value BAT54 -> PMEG4005EJ; footprint Diode_SMD:D_SOD-123 -> Diode_SMD:D_SOD-323F
- U1: footprint Package_LGA:Bosch_LGA-14_3x2.5mm_P0.5mm -> Kingfisher:ICM-45686
Connections:
- net +3V3: now also C1.1, C2.1, C3.1, C4.1, J1.1 (Pin_1), J1.17 (Pin_17), U1.12 (AP_CS), U1.5 (VDDIO), U1.8 (VDD), U2.1 (VDDIO), U2.10 (VDD), U2.6 (CSB), U5.7 (VDD), C11.1, J3.1 (Pin_1), R7.1, R8.1, TP1.1; no longer U1.3 (NC), U1.6 (GND), U2.3 (VSS), U2.4 (SDI), U2.8 (VSS)
- net +3V3_GPS: now also C6.1, C7.1, C8.1, D1.2 (A), U3.5 (VOUT), U4.23 (VCC), U4.7 (VDD_USB), R3.1, R6.1, TP3.1
- net +5V: now also C5.1, J1.2 (Pin_2), J1.4 (Pin_4), U3.1 (VIN), U3.3 (EN), TP2.1
- net GND: now also BT1.2 (-), C1.2, C2.2, C3.2, C4.2, C5.2, C6.2, C7.2, C8.2, J1.14 (Pin_14), J1.20 (Pin_20), J1.25 (Pin_25), J1.30 (Pin_30), J1.34 (Pin_34), J1.39 (Pin_39), J1.6 (Pin_6), J1.9 (Pin_9), J2.2 (Ext), U1.1 (AP_AD0), U1.6 (GND), U2.3 (VSS), U2.8 (VSS), U2.9 (VSS), U3.2 (GND), U4.10 (GND), U4.12 (GND), U4.13 (GND), U4.24 (GND), U5.5 (VSS), BT2.2 (-), C10.2, C11.2, C9.2, D2.1 (K), J3.2 (Pin_2), TP12.1; no longer U1.14 (AP_SDA), U1.5 (VDDIO), U2.1 (VDDIO), U2.10 (VDD)
- net GPS_PPS: now also J1.12 (Pin_12), U4.3 (TIMEPULSE), TP10.1
- net IMU_INT: now also J1.11 (Pin_11), U1.4 (INT1), TP11.1
- net SCL: now also J1.5 (Pin_5), U1.13 (AP_SCL), U2.2 (SCK), U5.3 (SCL), J3.4 (Pin_4), R8.2, TP7.1; no longer U1.2 (NC)
- net SDA: now also J1.3 (Pin_3), U1.14 (AP_SDA), U2.4 (SDI), U5.4 (SDA), J3.3 (Pin_3), R7.2, TP6.1; no longer U1.1 (AP_AD0), U2.6 (CSB), U5.8 (EVI)
- net UART_RX: now also J1.10 (Pin_10), R2.2, TP9.1
- net UART_TX: now also J1.8 (Pin_8), R1.1, TP8.1
- net VBAT: now also BT1.1 (+), U5.6 (VBACKUP), TP5.1
- net V_BCKP: now also U4.22 (V_BCKP), BT2.1 (+), C9.1, R4.2, TP4.1
- net CHG: now reaches D1.1 (K)
- net CHG: now also R4.1
- net PLD: now reaches J1.31 (Pin_31)
- net PLD: now also J3.5 (Pin_5)
- net RF: now reaches U4.11 (RF_IN)
- net RF: now also J2.1 (In), FB1.1
- net D_SEL: now reaches U4.2 (D_SEL)
- net D_SEL: now also R3.2
- net GPS_TX: now reaches U4.20 (TXD/SPI_MISO)
- net GPS_TX: now also R2.1
- net GPS_RX: now reaches U4.21 (RXD/SPI_MOSI)
- net GPS_RX: now also R1.2
- net VCC_RF: now reaches U4.9 (VCC_RF)
- net VCC_RF: now also R5.1
- new net BIAS: C10.1, FB1.2, R5.2
- new net LED_A: D2.2 (A), R6.2
- no-connect marks 0 -> 43
Other:
- note added: "Antenna bias: VCC_RF, 33 ohm, 47pF to GND, 120R ferrite onto RF_IN. Ferrite is the bias choke, not in series with the RF path and not on VCC."
- note added: "GPS backup is ML414H directly on V_BCKP, charged from +3V3_GPS through PMEG4005EJ and 1k. CR2032 feeds only RV-3028 VBACKUP."
- note added: "ICM-45686 0x68, BMP581 0x47, RV-3028-C7 0x52, NEO-M9N UART+PPS. No UPS."
- note added: "J3 X1200 harness, pin 1 to 5: +3V3, GND, SDA, SCL, GPIO6. R7 and R8 I2C pull-ups are DNP."
- note added: "Kingfisher Sensor HAT rev 0.3"
- note removed: "BT1 CR2032 RTC + GPS backup (primary, not charged)"
- note removed: "ICM-45686 + BMP581 + NEO-M9N + RV-3028 RTC + CR2032 backup"
- note removed: "Kingfisher Sensor HAT rev 0.2"
- note removed: "NOTES: ICM 0x68 / BMP581 0x47 / RV-3028 0x52 / UPS 0x36. CR2032 is primary — diode-OR must not charge it. Open in eeschema to tidy pin-label geometry before fab. See docs/DESIGN.md."
- note removed: "U1 ICM-45686 I2C 0x68 (AP_AD0=GND)"
- note removed: "U2 BMP581 I2C 0x47 (SDO=1)"
- note removed: "U3 AP2112K-3.3 GPS rail from +5V"
- note removed: "U4 NEO-M9N V_BCKP = diode-OR(+3V3_GPS, VBAT)"
- note removed: "U5 RV-3028-C7 I2C 0x52 VBACKUP=VBAT"
